File: AIO_tracker_V1.0.sch (EAGLE design)
At the start: 76 parts, among them IC1 TPS61201, IC2 TPS61201, J1 EDGE_ICSP, Q1 MOSFET-PCHANNELSMD, U1 ATMEGA328P-AU, U2 USD-SOCKETNEW, X1 SMA-142-0701-881/886, Y1 ABRACON_ABM3_CRYSTAL

Commit message: Final without logo
Parts:
- removed JP1: M02PTH, SparkFun-Connectors:M02PTH
- removed SJ2: SOLDERJUMPERNO, SparkFun-Passives:SOLDERJUMPERNO
- added CUTOFF: M021X02_NO_SILK, SparkFun-Connectors:M021X02_NO_SILK
- I2C: device SparkFun-Connectors:M05PTH -> SparkFun-Connectors:M05NO_SILK
- U$3: value RADIOMETRIX-HX1 -> NTX2-VERTICAL; device Ava:RADIOMETRIX-HX1 -> Ava:NTX2-VERTICAL
Connections:
- removed net N$8: C4.1, SJ2.1
- new net N$9: TP11.TP, TP12.TP
- net 3.3V: now also C4.1; no longer SJ2.2
- net CUTOUT: now also CUTOFF.2; no longer JP1.2
- net GND: now also CUTOFF.1; no longer JP1.1
- net N$25: no longer TP11.TP, TP12.TP
Changed lines of the file:
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@@
 <classes>
 <class number="0" name="default" width="0.254" drill="0.6">
-<clearance class="0" value="0.3048"/>
+<clearance class="0" value="0.254"/>
+</class>
+<class number="1" name="bat" width="0.8128" drill="0.6">
+<clearance class="1" value="0.4064"/>
+</class>
+<class number="2" name="5V" width="0.3048" drill="0.6">
+<clearance class="2" value="0.3048"/>
+</class>
+<class number="3" name="3.3V" width="0.3048" drill="0.6">
+<clearance class="3" value="0.3048"/>
+</class>
+<class number="4" name="GND" width="0.4064" drill="0.6">
+<clearance class="4" value="0.4064"/>
 </class>
 </classes>
@@
 <part name="U$1" library="Ava" deviceset="UBLOX_MAX-6" device=""/>
 <part name="U1" library="Ava" deviceset="ATMEGA328P-AU" device="" value=""/>
-<part name="U$3" library="Ava" deviceset="RADIOMETRIX-HX1" device=""/>
+<part name="U$3" library="Ava" deviceset="NTX2-VERTICAL" device=""/>
 <part name="R1" library="SparkFun-Passives" deviceset="RESISTOR" device="0603-RES" value="100k"/>
 <part name="Q1" library="SparkFun-DiscreteSemi" deviceset="MOSFET-PCHANNEL" device="SMD"/>
@@
 <part name="SUPPLY17" library="SparkFun-Aesthetics" deviceset="3.3V" device=""/>
 <part name="R14" library="SparkFun-Passives" deviceset="RESISTOR" device="0603-RES" value="4.7k"/>
-<part name="I2C" library="SparkFun-Connectors" deviceset="M05" device="PTH"/>
+<part name="I2C" library="SparkFun-Connectors" deviceset="M05" device="NO_SILK"/>
 <part name="SUPPLY20" library="SparkFun-Aesthetics" deviceset="5V" device=""/>
 <part name="SUPPLY21" library="SparkFun-Aesthetics" deviceset="3.3V" device=""/>
@@
 <part name="X1" library="con-coax" deviceset="SMA-" device="142-0701-881/886"/>
 <part name="VBATT" library="SparkFun-Connectors" deviceset="M01" device="SMDNS" value="M01SMDNS"/>
-<part name="SJ2" library="SparkFun-Passives" deviceset="SOLDERJUMPER" device="NO"/>
 <part name="U3" library="SparkFun-Sensors" deviceset="MPU-9150" device="QFN-24-NP"/>
 <part name="C14" library="SparkFun-Passives" deviceset="CAP" device="0603-CAP" value="2.2nF"/>
@@
 <part name="TP14" library="testpad" deviceset="TP" device="TP10SQ" value="TPTP10SQ"/>
 <part name="U$5" library="SparkFun-PowerIC" deviceset="LM2931_FIXED" device=""/>
-<part name="JP1" library="SparkFun-Connectors" deviceset="M02" device="PTH"/>
+<part name="CUTOFF" library="SparkFun-Connectors" deviceset="M02" device="1X02_NO_SILK" value="M021X02_NO_SILK"/>
 <part name="GND26" library="SparkFun-Aesthetics" deviceset="GND" device=""/>
 </parts>
@@
 <attribute name="NAME" x="137.16" y="-4.318" size="1.778" layer="95"/>
 </instance>
-<instance part="SJ2" gate="1" x="-35.56" y="-10.16" rot="R90"/>
 <instance part="U3" gate="G$1" x="-109.22" y="-48.26"/>
 <instance part="C14" gate="G$1" x="-139.7" y="-53.34"/>
@@
 <instance part="TP14" gate="G$1" x="-147.32" y="2.54"/>
 <instance part="U$5" gate="G$1" x="-91.44" y="58.42"/>
-<instance part="JP1" gate="G$1" x="-154.94" y="58.42"/>
+<instance part="CUTOFF" gate="G$1" x="-154.94" y="58.42"/>
 <instance part="GND26" gate="1" x="-142.24" y="55.88"/>
 </instances>
@@
 </busses>
 <nets>
-<net name="3.3V" class="0">
+<net name="3.3V" class="3">
 <segment>
 <pinref part="Q1" gate="G$1" pin="S"/>
@@
 <wire x1="-25.4" y1="7.62" x2="-25.4" y2="-5.08" width="0.1524" layer="91"/>
 <wire x1="-25.4" y1="-5.08" x2="-35.56" y2="-5.08" width="0.1524" layer="91"/>
-<pinref part="SJ2" gate="1" pin="2"/>
+<pinref part="C4" gate="G$1" pin="1"/>
+<wire x1="-35.56" y1="-17.78" x2="-35.56" y2="-5.08" width="0.1524" layer="91"/>
+<junction x="-25.4" y="-5.08"/>
 </segment>
 <segment>
@@
 <wire x1="-129.54" y1="-33.02" x2="-129.54" y2="-27.94" width="0.1524" layer="91"/>
 <pinref part="SUPPLY3" gate="G$1" pin="3.3V"/>
+<junction x="-129.54" y="-35.56"/>
+<junction x="-129.54" y="-33.02"/>
 </segment>
 <segment>
@@
 <label x="-139.7" y="30.48" size="1.778" layer="95"/>
 <pinref part="SUPPLY5" gate="G$1" pin="3.3V"/>
+<junction x="-134.62" y="30.48"/>
 </segment>
 </net>
@@
 </segment>
 </net>
-<net name="GND" class="0">
+<net name="GND" class="4">
 <segment>
 <pinref part="J1" gate="G$1" pin="6"/>
@@
 <label x="-154.94" y="30.48" size="1.778" layer="95"/>
 <pinref part="GND30" gate="1" pin="GND"/>
-</segment>
-<segment>
-<pinref part="JP1" gate="G$1" pin="1"/>
+<junction x="-149.86" y="30.48"/>
+</segment>
+<segment>
+<pinref part="CUTOFF" gate="G$1" pin="1"/>
 <wire x1="-147.32" y1="58.42" x2="-142.24" y2="58.42" width="0.1524" layer="91"/>
 <pinref part="GND26" gate="1" pin="GND"/>
@@
 <wire x1="-149.86" y1="20.32" x2="-154.94" y2="20.32" width="0.1524" layer="91"/>
 <label x="-154.94" y="20.32" size="1.778" layer="95"/>
+<junction x="-149.86" y="20.32"/>
 </segment>
 </net>
@@
 <wire x1="-134.62" y1="20.32" x2="-139.7" y2="20.32" width="0.1524" layer="91"/>
 <label x="-139.7" y="20.32" size="1.778" layer="95"/>
+<junction x="-134.62" y="20.32"/>
 </segment>
 </net>
@@
 <wire x1="-17.78" y1="-45.72" x2="-17.78" y2="-48.26" width="0.1524" layer="91"/>
 <wire x1="-12.7" y1="-48.26" x2="-17.78" y2="-48.26" width="0.1524" layer="91"/>
+<junction x="-17.78" y="-48.26"/>
 </segment>
 </net>
@@
 <wire x1="-17.78" y1="-40.64" x2="-17.78" y2="-38.1" width="0.1524" layer="91"/>
 <wire x1="-12.7" y1="-38.1" x2="-17.78" y2="-38.1" width="0.1524" layer="91"/>
-</segment>
-</net>
-<net name="VBATT" class="0">
+<junction x="-17.78" y="-38.1"/>
+</segment>
+</net>
+<net name="VBATT" class="1">
 <segment>
 <wire x1="-30.48" y1="66.04" x2="-22.86" y2="66.04" width="0.1524" layer="91"/>
@@
 </segment>
 </net>
-<net name="5V" class="0">
+<net name="5V" class="2">
 <segment>
 <wire x1="99.06" y1="71.12" x2="99.06" y2="66.04" width="0.1524" layer="91"/>
@@
 </segment>
 </net>
-<net name="N$8" class="0">
-<segment>
-<pinref part="C4" gate="G$1" pin="1"/>
-<pinref part="SJ2" gate="1" pin="1"/>
-<wire x1="-35.56" y1="-17.78" x2="-35.56" y2="-15.24" width="0.1524" layer="91"/>
-</segment>
-</net>
 <net name="N$17" class="0">
 <segment>
@@
 </net>
 <net name="N$25" class="0">
-<segment>
-<pinref part="TP12" gate="G$1" pin="TP"/>
-<pinref part="TP11" gate="G$1" pin="TP"/>
-<wire x1="-132.08" y1="10.16" x2="-134.62" y2="10.16" width="0.1524" layer="91"/>
-<wire x1="-134.62" y1="10.16" x2="-139.7" y2="10.16" width="0.1524" layer="91"/>
-<label x="-139.7" y="10.16" size="1.778" layer="95"/>
-</segment>
 <segment>
 <pinref part="TP10" gate="G$1" pin="TP"/>
@@
 <wire x1="-149.86" y1="10.16" x2="-154.94" y2="10.16" width="0.1524" layer="91"/>
 <label x="-154.94" y="10.16" size="1.778" layer="95"/>
-</segment>
-</net>
-<net name="N$9" class="0">
-<segment>
-<pinref part="TP16" gate="G$1" pin="TP"/>
-<pinref part="TP15" gate="G$1" pin="TP"/>
-<wire x1="-132.08" y1="0" x2="-134.62" y2="0" width="0.1524" layer="91"/>
-<wire x1="-134.62" y1="0" x2="-139.7" y2="0" width="0.1524" layer="91"/>
-</segment>
-</net>
-<net name="N$14" class="0">
-<segment>
-<pinref part="TP14" gate="G$1" pin="TP"/>
-<pinref part="TP13" gate="G$1" pin="TP"/>
-<wire x1="-147.32" y1="0" x2="-149.86" y2="0" width="0.1524" layer="91"/>
-<wire x1="-149.86" y1="0" x2="-154.94" y2="0" width="0.1524" layer="91"/>
+<junction x="-149.86" y="10.16"/>
 </segment>
 </net>
@@
 </segment>
 <segment>
-<pinref part="JP1" gate="G$1" pin="2"/>
+<pinref part="CUTOFF" gate="G$1" pin="2"/>
 <wire x1="-147.32" y1="60.96" x2="-142.24" y2="60.96" width="0.1524" layer="91"/>
 <label x="-144.78" y="60.96" size="1.778" layer="95"/>
@@
 </segment>
 </net>
+<net name="N$9" class="0">
+<segment>
+<pinref part="TP12" gate="G$1" pin="TP"/>
+<wire x1="-132.08" y1="10.16" x2="-134.62" y2="10.16" width="0.1524" layer="91"/>
+<label x="-139.7" y="10.16" size="1.778" layer="95"/>
+<pinref part="TP11" gate="G$1" pin="TP"/>
+<wire x1="-134.62" y1="10.16" x2="-139.7" y2="10.16" width="0.1524" layer="91"/>
+<junction x="-134.62" y="10.16"/>
+</segment>
+</net>
+<net name="N$14" class="0">
+<segment>
+<pinref part="TP16" gate="G$1" pin="TP"/>
+<wire x1="-132.08" y1="0" x2="-134.62" y2="0" width="0.1524" layer="91"/>
+<label x="-139.7" y="0" size="1.778" layer="95"/>
+<pinref part="TP15" gate="G$1" pin="TP"/>
+<wire x1="-134.62" y1="0" x2="-139.7" y2="0" width="0.1524" layer="91"/>
+<junction x="-134.62" y="0"/>
+</segment>
+</net>
+<net name="N$23" class="0">
+<segment>
+<pinref part="TP14" gate="G$1" pin="TP"/>
+<wire x1="-147.32" y1="0" x2="-149.86" y2="0" width="0.1524" layer="91"/>
+<label x="-154.94" y="0" size="1.778" layer="95"/>
+<pinref part="TP13" gate="G$1" pin="TP"/>
+<wire x1="-149.86" y1="0" x2="-154.94" y2="0" width="0.1524" layer="91"/>
+<junction x="-149.86" y="0"/>
+</segment>
+</net>

Commit message: corrected last things
Parts:
- U$4, U$6: value COILCRAFT-MSS5131 -> 2.2uH
Other:
- note added: "3V3_VReg"
- note added: "5V_VReg"
- note added: "9DOF"
- note added: "AA_Battery"
- note added: "APRS"
- note added: "ATMEGA 328"
- note added: "Cutoff Pins"
- note added: "Cutoff_Mosfet"
- note added: "I2C Pins"
- note added: "ICSP Program"
- note added: "LED"
- note added: "Power Pins"
- note added: "Pressure"
- note added: "RTTY"
- note added: "RX_TX"
- note added: "Soft_Serial"
- note added: "Temperature"
- note added: "UBlox_GPS"
- note added: "Voltage"
- note added: "uSD Socket"
- moved on the sheet: 3.3V, 5V, BAT1, BAT2, C1, C10, C11, C12, C13, C14, C15, C2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
