File: AIO_tracker_V1.0.brd (EAGLE design)
At the start: 60 x 55 mm, 75 parts, among them J1 EDGE_ICSP, Q1 MOSFET-PCHANNELSMD, U2 USD-SOCKETNEW, X1 SMA-142-0701-881/886, Y1 ABRACON_ABM3_CRYSTAL

Commit message: corrected last things
Parts:
- U$4, U$6: value COILCRAFT-MSS5131 -> 2.2uH
Changed lines of the file:
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@@
 <attribute name="NAME" x="6.638" y="14.761" size="0.4064" layer="25" font="vector" ratio="25" rot="R90"/>
 </element>
-<element name="U$4" library="Ava" package="COILCRAFT_MSS5131" value="COILCRAFT-MSS5131" x="23.75" y="3.78" smashed="yes" rot="R270"/>
-<element name="U$6" library="Ava" package="COILCRAFT_MSS5131" value="COILCRAFT-MSS5131" x="33.4" y="3.78" smashed="yes" rot="R270"/>
+<element name="U$4" library="Ava" package="COILCRAFT_MSS5131" value="2.2uH" x="23.75" y="3.78" smashed="yes" rot="R270"/>
+<element name="U$6" library="Ava" package="COILCRAFT_MSS5131" value="2.2uH" x="33.4" y="3.78" smashed="yes" rot="R270"/>
 <element name="JP5" library="SparkFun-Connectors" package="1X01" value="M01PTH" x="18.4" y="34.4" smashed="yes" rot="R180"/>
 <element name="JP6" library="SparkFun-Connectors" package="1X01" value="M01PTH" x="21.3" y="34.4" smashed="yes" rot="R180"/>
@@
 <wire x1="-1.515" y1="37.54" x2="-2.531" y2="37.54" width="0.4064" layer="16"/>
 </signal>
+<signal name="N$8">
+</signal>
 </signals>

Commit message: final commit of pcb (fingers crossed)
Parts:
- moved C3 0.10 mm to (8.40, 14.8)
Other:
- board text added: "All-In-One HAB Tracker"
- board text added: "V2.0"
- board text removed: "All-In-One HAB Tracker V2.0"
Changed lines of the file:
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@@
 <wire x1="47" y1="39" x2="-13" y2="39" width="0" layer="20"/>
 <wire x1="-13" y1="39" x2="-13" y2="-16" width="0" layer="20"/>
-<text x="9.3" y="-14.2" size="1.27" layer="25" font="vector" ratio="16" distance="0" rot="SR0">BALUA.ORG</text>
-<text x="7.1" y="-15.3" size="0.6096" layer="25" font="vector" ratio="25" rot="SR0">All-In-One HAB Tracker V2.0</text>
+<text x="12.3" y="-13.4" size="1.4224" layer="25" font="vector" ratio="16" distance="0" rot="SR0">BALUA.ORG</text>
+<text x="10.6" y="-14.9" size="0.6096" layer="25" font="vector" ratio="25" rot="SR0">All-In-One HAB Tracker</text>
 <text x="22.6" y="36.35" size="0.4064" layer="25" font="vector" ratio="25" rot="R180">Soft_Serial A3-A2</text>
 <text x="43.4" y="2.2" size="0.4064" layer="25" font="vector" ratio="25" distance="25" rot="R90">VBatt</text>
@@
 <hole x="45" y="-14" drill="2.5"/>
 <hole x="45" y="36" drill="2.5"/>
-<text x="21" y="-15.3" size="0.6096" layer="26" font="vector" ratio="25" rot="SMR0">All-In-One HAB Tracker V2.0</text>
-<text x="19" y="-14.2" size="1.27" layer="26" font="vector" ratio="16" distance="0" rot="SMR0">BALUA.ORG</text>
+<text x="25.7" y="-14.9" size="0.6096" layer="26" font="vector" ratio="25" rot="SMR0">All-In-One HAB Tracker</text>
+<text x="23.1" y="-13.4" size="1.4224" layer="26" font="vector" ratio="16" distance="0" rot="SMR0">BALUA.ORG</text>
+<text x="8.6" y="-9.4" size="1.778" layer="25"> V2.0</text>
+<text x="8.6" y="-9.4" size="1.778" layer="25"> V2.0</text>
+<text x="21.7" y="-14.9" size="1.016" layer="25" font="vector" ratio="25"> V2.0</text>
+<text x="14.6" y="-14.9" size="1.016" layer="26" font="vector" ratio="25" rot="MR0"> V2.0</text>
 </plain>
 <attributes>
@@
 <attribute name="NAME" x="8.261" y="23.462" size="0.4064" layer="25" font="vector" ratio="25"/>
 </element>
-<element name="C3" library="SparkFun-Passives" package="0603-CAP" value="18pF" x="8.4" y="14.9" smashed="yes">
-<attribute name="NAME" x="6.638" y="14.761" size="0.4064" layer="25" font="vector" ratio="25" rot="R90"/>
+<element name="C3" library="SparkFun-Passives" package="0603-CAP" value="18pF" x="8.4" y="14.8" smashed="yes">
+<attribute name="NAME" x="6.638" y="14.661" size="0.4064" layer="25" font="vector" ratio="25" rot="R90"/>
 </element>
 <element name="U$4" library="Ava" package="COILCRAFT_MSS5131" value="2.2uH" x="23.75" y="3.78" smashed="yes" rot="R270"/>
@@
 <via x="3.79" y="37.7865" extent="1-16" drill="0.5" diameter="0.4064"/>
 <wire x1="7.5" y1="15.15" x2="7.5" y2="14.95" width="0.4064" layer="1"/>
-<wire x1="7.5" y1="14.95" x2="7.55" y2="14.9" width="0.4064" layer="1"/>
+<wire x1="7.5" y1="14.95" x2="7.55" y2="14.8" width="0.4064" layer="1"/>
 </signal>
 <signal name="N$4">
@@
 <wire x1="13.5" y1="18.1" x2="13.5182" y2="18.146" width="0.254" layer="1"/>
 <wire x1="9.2" y1="16.65" x2="9.1" y2="16.6" width="0.254" layer="1"/>
-<wire x1="9.25" y1="14.9" x2="9.1" y2="15.05" width="0.254" layer="1"/>
+<wire x1="9.25" y1="14.8" x2="9.1" y2="15.05" width="0.254" layer="1"/>
 <wire x1="9.1" y1="15.05" x2="9.1" y2="16.6" width="0.254" layer="1"/>
 </signal>

Commit message: Several thing corrected (still....=/)
Position of 9DOF, tended vias, names, etc
Parts:
- U$1: value UBLOX_MAX-6 -> UBLOX_MAX; device Ava:UBLOX_MAX-6 -> Ava:UBLOX_MAX
- moved C14 57.7 mm to (44.4, 32.8), turned to 0 degrees
- moved U3 56.2 mm to (41.0, 27.3)
- moved C15 56.0 mm to (40.3, 23.2), turned to 180 degrees
- moved C4 31.3 mm to (-6.90, -0.80), turned to 270 degrees
- moved C1 2.02 mm to (25.8, 8.20)
- moved C10 1.84 mm to (28.0, 8.20)
- moved R6 1.43 mm to (24.3, 10.7), turned to 180 degrees
- moved LED1 0.94 mm to (16.4, 8.00), turned to 90 degrees
- moved U$5 0.61 mm to (38.7, 10.7)
- moved R2 0.34 mm to (-10.1, 23.5)
- moved C5 0.28 mm to (28.3, 13.7)
Routing:
- net SDA: track 219.2 -> 85.0 mm, vias 11 -> 6
- net SCL: track 168.8 -> 106.6 mm, vias 10 -> 6
- net GND: track 100.6 -> 84.7 mm, vias 132 -> 134
- net 3.3V: track 212.2 -> 217.0 mm
- net MISO: track 57.6 -> 54.6 mm
- net VBATTADC: track 20.9 -> 18.6 mm
- net MOSI: track 56.0 -> 58.1 mm
- net GPSEN: track 31.5 -> 33.1 mm
- net RESET: track 43.9 -> 45.2 mm
- net VBATT: track 89.1 -> 88.1 mm
- net N$15: track 13.8 -> 14.4 mm
